Commit message: good loading for zoey - scale missin

File: Zoey/human.urdf (robot description, URDF)
Before this commit: robot human, 43 links, 42 joints
Links:
- removed link head_endeffector_link
- added link torso_up_link
- link lower_right_leg_link: geometry collision mesh filename=../Zoey/r_lowerleg.obj; visual mesh filename=../Zoey/r_lowerleg.obj
- link upper_right_arm_x_link: geometry collision mesh filename=../Zoey/r_upperarm.obj; visual mesh filename=../Zoey/r_upperarm.obj
Joints:
- removed joint head_endeffector_joint
- added joint torso_up_joint: type revolute, parent torso_x_link, child torso_up_link, origin xyz=0 -0.5594 6.5653 rpy=0 0 0, axis 1 0 0, limit lower=-0.001 upper=0.001 effort=15 velocity=5
- joint head_z_joint: origin xyz=0 17 -2 rpy=0 0 0 -> xyz=0 -1.55  10.8489 rpy=0 0 0; parent torso_x_link -> torso_up_link
- joint left_foot_z_joint: origin xyz=-0.5707  -16.2423  -0.6640 rpy=0 0 0 -> xyz=0.5707 -0.6640 -16.2423 rpy=0 0 0
- joint left_hand_endeffector_joint: origin xyz= 0.3487 -4.4781 0.0080 rpy=0 0 0 -> xyz= -0.3487 0.0080  -4.4781 rpy=0 0 0
- joint left_hand_z_joint: origin xyz=6.4684 -19.7609  2.2908 rpy=0 0 0 -> xyz= -3.0173 1.7858  -9.2177 rpy=0 0 0
- joint lower_left_arm_joint: origin xyz= 3.4512 -10.5432 0.5050 rpy=0 0 0 -> xyz= -3.4512 0.5050 -10.5432 rpy=0 0 0
- joint lower_left_leg_joint: origin xyz=-6.3295 -16.5541 -0.5126 rpy=0 0 0 -> xyz=0.5817 -0.5126 -16.5541 rpy=0 0 0
- joint lower_right_arm_joint: origin xyz= -3.4512 -10.5432 0.5051 rpy=0 0 0 -> xyz= 3.4512 0.5051 -10.5432 rpy=0 0 0
- joint lower_right_leg_joint: origin xyz=0.5817 -16.5541 -0.5226 rpy=0 0 0 -> xyz=-0.5817 -0.5226 -16.5541 rpy=0 0 0
- joint right_foot_z_joint: origin xyz= 0.5707  -16.2423 -0.6640 rpy=0 0 0 -> xyz=-0.5707 -0.6640 -16.2423 rpy=0 0 0
- joint right_hand_endeffector_joint: origin xyz=-0.5536 -4.9991  0.8500 rpy=0 0 0 -> xyz=0.5536 0.8500 -4.9991 rpy=0 0 0
- joint right_hand_z_joint: origin xyz=-3.0174 -9.2177 1.7858 rpy=0 0 0 -> xyz=3.0174 1.7858  -9.2177 rpy=0 0 0
- joint torso_z_joint: origin xyz=0 3.7037 0.2932 rpy=0 0 0 -> xyz=0 0.2932 3.7037 rpy=0 0 0
- joint upper_left_arm_z_joint: origin xyz= 3.7479 -1.6899 -1.3488 rpy=0 0 0 -> xyz= -3.7479 -1.3488 -1.6899 rpy=0 0 0
- joint upper_left_leg_z_joint: origin xyz=3.4556 0 0 rpy=0 0 0 -> xyz=-3.4556 0 0 rpy=0 0 0
- joint upper_left_specula_joint: origin xyz= 1.5000 16.1163 -0.7763 rpy=0 0 0 -> xyz= -1.5000 -0.2170  9.5510 rpy=0 0 0; parent torso_x_link -> torso_up_link
- joint upper_right_arm_z_joint: origin xyz=-3.7478 -1.6900 -1.3488 rpy=0 0 0 -> xyz=3.7478 -1.3488  -1.6900 rpy=0 0 0
- joint upper_right_leg_z_joint: origin xyz=-3.4556 0 0.01 rpy=0 0 0 -> xyz=3.4556 0 0 rpy=0 0 0
- joint upper_right_specula_joint: origin xyz= -1.5000 16.1163 -0.7763 rpy=0 0 0 -> xyz= 1.5000 -0.2170  9.5510 rpy=0 0 0; parent torso_x_link -> torso_up_link
