Commit message: zoe urdf

File: zoe.urdf (robot description, URDF)
Before this commit: robot human, 43 links, 42 joints
Links:
- removed link torso_up_link
- removed link upper_left_arm_specula_link
- removed link upper_right_arm_specula_link
- added link head_endeffector_link; collision box size=0.001 0.001 0.001; visual box size=0.001 0.001 0.001
- link head_x_link: geometry collision mesh filename=../humandes/head.obj; visual mesh filename=../humandes/head.obj
- link left_foot_x_link: geometry collision mesh filename=../humandes/leftFoot.obj; visual mesh filename=../humandes/leftFoot.obj
- link left_hand_x_link: geometry collision mesh filename=../humandes/leftHand.obj; visual mesh filename=../humandes/leftHand.obj
- link lower_left_arm_link: geometry collision mesh filename=../humandes/lowerLeftArm.obj; visual mesh filename=../humandes/lowerLeftArm.obj
- link lower_left_leg_link: geometry collision mesh filename=../humandes/lowerLeftLeg.obj; visual mesh filename=../humandes/lowerLeftLeg.obj
- link lower_right_arm_link: geometry collision mesh filename=../humandes/lowerRightArm.obj; visual mesh filename=../humandes/lowerRightArm.obj
- link lower_right_leg_link: geometry collision mesh filename=../humandes/lowerRightLeg.obj; visual mesh filename=../humandes/lowerRightLeg.obj
- link pelvis_link: geometry collision mesh filename=../humandes/pelvis.obj; visual mesh filename=../humandes/pelvis.obj
- link right_foot_x_link: geometry collision mesh filename=../humandes/rightFoot.obj; visual mesh filename=../humandes/rightFoot.obj
- link right_hand_x_link: geometry collision mesh filename=../humandes/rightHand.obj; visual mesh filename=../humandes/rightHand.obj
- link torso_x_link: geometry collision mesh filename=../humandes/torso.obj; visual mesh filename=../humandes/torso.obj
- link upper_left_arm_x_link: geometry collision mesh filename=../humandes/upperLeftArm.obj; visual mesh filename=../humandes/upperLeftArm.obj
- link upper_left_leg_x_link: geometry collision mesh filename=../humandes/upperLeftLeg.obj; visual mesh filename=../humandes/upperLeftLeg.obj
- link upper_right_arm_x_link: geometry collision mesh filename=../humandes/upperRightArm.obj; visual mesh filename=../humandes/upperRightArm.obj
- link upper_right_leg_x_link: geometry collision mesh filename=../humandes/upperRightLeg.obj; visual mesh filename=../humandes/upperRightLeg.obj
Joints:
- removed joint torso_up_joint
- removed joint upper_left_specula_joint
- removed joint upper_right_specula_joint
- added joint head_endeffector_joint: type revolute, parent head_x_link, child head_endeffector_link, origin xyz=0 0 0.3 rpy=0 0 0, axis 0 0 1, limit lower=-0.001 upper=0.001 effort=15 velocity=5
- joint head_z_joint: origin xyz=0 -0.031 0.216978 rpy=0 0 0 -> xyz=0 0 0.45 rpy=0 0 0; parent torso_up_link -> torso_x_link
- joint left_foot_z_joint: origin xyz=0.011414 -0.01328 -0.324846 rpy=0 0 0 -> xyz=0 0 -0.52 rpy=0 0 0
- joint left_hand_endeffector_joint: origin xyz=-0.006974 0.00016 -0.089562 rpy=0 0 0 -> xyz=0 0 -0.2 rpy=0 0 0
- joint left_hand_z_joint: origin xyz=-0.060346 0.035716 -0.184354 rpy=0 0 0 -> xyz=0 0 -0.35 rpy=0 0 0
- joint lower_left_arm_joint: origin xyz=-0.069024 0.0101 -0.210864 rpy=0 0 0 -> xyz=0 0 -0.35 rpy=0 0 0
- joint lower_left_leg_joint: origin xyz=0.011634 -0.010252 -0.331082 rpy=0 0 0 -> xyz=0 0 -0.5 rpy=0 0 0
- joint lower_right_arm_joint: origin xyz=0.069024 0.010102 -0.210864 rpy=0 0 0 -> xyz=0 0 -0.35 rpy=0 0 0
- joint lower_right_leg_joint: origin xyz=-0.011634 -0.010452 -0.331082 rpy=0 0 0 -> xyz=0 0 -0.5 rpy=0 0 0
- joint right_foot_z_joint: origin xyz=-0.011414 -0.01328 -0.324846 rpy=0 0 0 -> xyz=0 0 -0.52 rpy=0 0 0
- joint right_hand_endeffector_joint: origin xyz=0.011072 0.017 -0.099982 rpy=0 0 0 -> xyz=0 0 -0.2 rpy=0 0 0
- joint right_hand_z_joint: origin xyz=0.060348 0.035716 -0.184354 rpy=0 0 0 -> xyz=0 0 -0.35 rpy=0 0 0
- joint torso_z_joint: origin xyz=0 0.005864 0.074074 rpy=0 0 0 -> xyz=0 0 0.26 rpy=0 0 0
- joint upper_left_arm_z_joint: origin xyz=-0.074958 -0.026976 -0.033798 rpy=0 0 0 -> xyz=-0.23 0 0.33 rpy=0 0 0; parent upper_left_arm_specula_link -> torso_x_link
- joint upper_left_leg_z_joint: origin xyz=-0.069112 0 0 rpy=0 0 0 -> xyz=-0.1 0 0 rpy=0 0 0
- joint upper_right_arm_z_joint: origin xyz=0.074956 -0.026976 -0.0338 rpy=0 0 0 -> xyz=0.23 0 0.33 rpy=0 0 0; parent upper_right_arm_specula_link -> torso_x_link
- joint upper_right_leg_z_joint: origin xyz=0.069112 0 0 rpy=0 0 0 -> xyz=0.1 0 0 rpy=0 0 0
