Commit message: added global rotation joint

File: spider/model/spider.urdf (robot description, URDF)
Before this commit: robot rocketbox_male, 37 links, 36 joints
Links:
- added link middleleftshoulder_link
Joints:
- added joint Shoulder_joint: type revolute, parent head_link, child middleleftshoulder_link, origin xyz=0 0 0 rpy=0 0 0, axis 0 0 1, limit lower=-1.57 upper=1 effort=15 velocity=5
- joint MiddleLeftUpperLimb_z_joint: parent head_link -> middleleftshoulder_link

Commit message: full spider model

File: spider/model/spider.urdf (robot description, URDF)
Before this commit: robot rocketbox_male, 38 links, 37 joints
Links:
- removed link left_foot_cp_1_link
- removed link left_foot_cp_2_link
- removed link left_foot_cp_3_link
- removed link left_foot_cp_4_link
- removed link left_foot_endeffector_link
- added link BackLeftEffector_x_link, mass 2.24629475115; collision mesh filename=../spider/model/mesh/MiddleLeftEffector.obj; visual mesh filename=../spider/model/mesh/MiddleLeftEffector.obj
- added link BackLeftEffector_y_link
- added link BackLeftEffector_z_link
- added link BackLeftLimb_link, mass 8.394054321; collision mesh filename=../spider/model/mesh/MiddleLeftLimb.obj; visual mesh filename=../spider/model/mesh/MiddleLeftLimb.obj
- added link BackLeftLowerLimb_link, mass 8.394054321; collision mesh filename=../spider/model/mesh/MiddleLeftLowerLimb.obj; visual mesh filename=../spider/model/mesh/MiddleLeftLowerLimb.obj
- added link BackLeftUpperLimb_x_link, mass 11.28066677275; collision mesh filename=../spider/model/mesh/MiddleLeftUpperLimb.obj; visual mesh filename=../spider/model/mesh/MiddleLeftUpperLimb.obj
- added link BackLeftUpperLimb_y_link
- added link BackLeftUpperLimb_z_link
- added link BackLeft_foot_cp_1_link, mass 0; visual box size=0.001 0.001 0.001
- added link BackLeft_foot_cp_2_link, mass 0; visual box size=0.001 0.001 0.001
- added link BackLeft_foot_cp_3_link, mass 0; visual box size=0.001 0.001 0.001
- added link BackLeft_foot_cp_4_link, mass 0; visual box size=0.001 0.001 0.001
- added link BackLeft_foot_endeffector_link; visual box size=0.001 0.001 0.001
- added link BackLeftshoulder_link
- added link BackRightEffector_x_link, mass 2.24629475115; collision mesh filename=../spider/model/mesh/MiddleLeftEffector.obj; visual mesh filename=../spider/model/mesh/MiddleLeftEffector.obj
- added link BackRightEffector_y_link
- added link BackRightEffector_z_link
- added link BackRightLimb_link, mass 8.394054321; collision mesh filename=../spider/model/mesh/MiddleLeftLimb.obj; visual mesh filename=../spider/model/mesh/MiddleLeftLimb.obj
- added link BackRightLowerLimb_link, mass 8.394054321; collision mesh filename=../spider/model/mesh/MiddleLeftLowerLimb.obj; visual mesh filename=../spider/model/mesh/MiddleLeftLowerLimb.obj
- added link BackRightUpperLimb_x_link, mass 11.28066677275; collision mesh filename=../spider/model/mesh/MiddleLeftUpperLimb.obj; visual mesh filename=../spider/model/mesh/MiddleLeftUpperLimb.obj
- added link BackRightUpperLimb_y_link
- added link BackRightUpperLimb_z_link
- added link BackRight_foot_cp_1_link, mass 0; visual box size=0.001 0.001 0.001
- added link BackRight_foot_cp_2_link, mass 0; visual box size=0.001 0.001 0.001
- added link BackRight_foot_cp_3_link, mass 0; visual box size=0.001 0.001 0.001
- added link BackRight_foot_cp_4_link, mass 0; visual box size=0.001 0.001 0.001
- added link BackRight_foot_endeffector_link; visual box size=0.001 0.001 0.001
- added link BackRightshoulder_link
- added link FrontRightEffector_x_link, mass 2.24629475115; collision mesh filename=../spider/model/mesh/MiddleLeftEffector.obj; visual mesh filename=../spider/model/mesh/MiddleLeftEffector.obj
- added link FrontRightEffector_y_link
- added link FrontRightEffector_z_link
- added link FrontRightLimb_link, mass 8.394054321; collision mesh filename=../spider/model/mesh/MiddleLeftLimb.obj; visual mesh filename=../spider/model/mesh/MiddleLeftLimb.obj
- added link FrontRightLowerLimb_link, mass 8.394054321; collision mesh filename=../spider/model/mesh/MiddleLeftLowerLimb.obj; visual mesh filename=../spider/model/mesh/MiddleLeftLowerLimb.obj
- added link FrontRightUpperLimb_x_link, mass 11.28066677275; collision mesh filename=../spider/model/mesh/MiddleLeftUpperLimb.obj; visual mesh filename=../spider/model/mesh/MiddleLeftUpperLimb.obj
- added link FrontRightUpperLimb_y_link
- added link FrontRightUpperLimb_z_link
- added link FrontRight_foot_cp_1_link, mass 0; visual box size=0.001 0.001 0.001
- added link FrontRight_foot_cp_2_link, mass 0; visual box size=0.001 0.001 0.001
- added link FrontRight_foot_cp_3_link, mass 0; visual box size=0.001 0.001 0.001
- added link FrontRight_foot_cp_4_link, mass 0; visual box size=0.001 0.001 0.001
- added link FrontRight_foot_endeffector_link; visual box size=0.001 0.001 0.001
- added link FrontRightshoulder_link
- added link Frontleft_foot_cp_1_link, mass 0; visual box size=0.001 0.001 0.001
- added link Frontleft_foot_cp_2_link, mass 0; visual box size=0.001 0.001 0.001
- added link Frontleft_foot_cp_3_link, mass 0; visual box size=0.001 0.001 0.001
- added link Frontleft_foot_cp_4_link, mass 0; visual box size=0.001 0.001 0.001
- added link Frontleft_foot_endeffector_link; visual box size=0.001 0.001 0.001
- added link MiddleRightEffector_x_link, mass 2.24629475115; collision mesh filename=../spider/model/mesh/MiddleLeftEffector.obj; visual mesh filename=../spider/model/mesh/MiddleLeftEffector.obj
- added link MiddleRightEffector_y_link
- added link MiddleRightEffector_z_link
- added link MiddleRightLimb_link, mass 8.394054321; collision mesh filename=../spider/model/mesh/MiddleLeftLimb.obj; visual mesh filename=../spider/model/mesh/MiddleLeftLimb.obj
- added link MiddleRightLowerLimb_link, mass 8.394054321; collision mesh filename=../spider/model/mesh/MiddleLeftLowerLimb.obj; visual mesh filename=../spider/model/mesh/MiddleLeftLowerLimb.obj
- added link MiddleRightUpperLimb_x_link, mass 11.28066677275; collision mesh filename=../spider/model/mesh/MiddleLeftUpperLimb.obj; visual mesh filename=../spider/model/mesh/MiddleLeftUpperLimb.obj
- added link MiddleRightUpperLimb_y_link
- added link MiddleRightUpperLimb_z_link
- added link MiddleRight_foot_cp_1_link, mass 0; visual box size=0.001 0.001 0.001
- added link MiddleRight_foot_cp_2_link, mass 0; visual box size=0.001 0.001 0.001
- added link MiddleRight_foot_cp_3_link, mass 0; visual box size=0.001 0.001 0.001
- added link MiddleRight_foot_cp_4_link, mass 0; visual box size=0.001 0.001 0.001
- added link MiddleRight_foot_endeffector_link; visual box size=0.001 0.001 0.001
- added link MiddleRightshoulder_link
- added link frontleftshoulder_link
- link FrontLeftEffector_x_link: geometry collision mesh filename=../spider/model/mesh/MiddleLeftEffector.obj; visual mesh filename=../spider/model/mesh/MiddleLeftEffector.obj
- link FrontLeftLimb_link: geometry collision mesh filename=../spider/model/mesh/MiddleLeftLimb.obj; visual mesh filename=../spider/model/mesh/MiddleLeftLimb.obj
- link FrontLeftLowerLimb_link: geometry collision mesh filename=../spider/model/mesh/MiddleLeftLowerLimb.obj; visual mesh filename=../spider/model/mesh/MiddleLeftLowerLimb.obj
- link FrontLeftUpperLimb_x_link: geometry collision mesh filename=../spider/model/mesh/MiddleLeftUpperLimb.obj; visual mesh filename=../spider/model/mesh/MiddleLeftUpperLimb.obj
Joints:
- removed joint Shoulder_joint
- removed joint left_foot_cp_1_joint
- removed joint left_foot_cp_2_joint
- removed joint left_foot_cp_3_joint
- removed joint left_foot_cp_4_joint
- removed joint left_foot_endeffector_joint
- added joint BackLeftEffector_x_joint: type revolute, parent BackLeftEffector_y_link, child BackLeftEffector_x_link, origin xyz=0 0 0 rpy=0 0 0, axis 1 0 0, limit lower=-0.8 upper=0.6 effort=15 velocity=5
- added joint BackLeftEffector_y_joint: type revolute, parent BackLeftEffector_z_link, child BackLeftEffector_y_link, origin xyz=0 0 0 rpy=0 0 0, axis 0 1 0, limit lower=-0.5 upper=0.5 effort=15 velocity=5
- added joint BackLeftEffector_z_joint: type revolute, parent BackLeftLowerLimb_link, child BackLeftEffector_z_link, origin xyz=-0.4343 -0.054 -0.1597 rpy=0 0 0, axis 0 0 1, limit lower=-0.01 upper=0 effort=15 velocity=5
- added joint BackLeftLimb_joint: type revolute, parent BackLeftUpperLimb_x_link, child BackLeftLimb_link, origin xyz=-0.4456 0.0015 0.1781 rpy=0 0 0, axis 0 1 0, limit lower=-2.4 upper=0 effort=15 velocity=5
- added joint BackLeftLowerLimb_joint: type revolute, parent BackLeftLimb_link, child BackLeftLowerLimb_link, origin xyz=-0.3928 -0.0167 -0.3044 rpy=0 0 0, axis 0 1 0, limit lower=-2.4 upper=0 effort=15 velocity=5
- added joint BackLeftUpperLimb_x_joint: type revolute, parent BackLeftUpperLimb_y_link, child BackLeftUpperLimb_x_link, origin xyz=0 0 0 rpy=0 0 0, axis 1 0 0, limit lower=-1.2 upper=1.57 effort=15 velocity=5
- added joint BackLeftUpperLimb_y_joint: type revolute, parent BackLeftUpperLimb_z_link, child BackLeftUpperLimb_y_link, origin xyz=0 0 0 rpy=0 0 0, axis 0 1 0, limit lower=-1.57 upper=0.7 effort=15 velocity=5
- added joint BackLeftUpperLimb_z_joint: type revolute, parent BackLeftshoulder_link, child BackLeftUpperLimb_z_link, origin xyz=-0.1891 0 -0.0795 rpy=0 0 0, axis 0 0 1, limit lower=-1.57 upper=1 effort=15 velocity=5
- added joint BackLeft_foot_cp_1_joint: type revolute, parent BackLeftEffector_x_link, child BackLeft_foot_cp_1_link, origin xyz=0.08027 0.27372 -0.12195 rpy=0 0 0, axis 0 0 1, limit lower=0 upper=0 effort=15 velocity=5
- added joint BackLeft_foot_cp_2_joint: type revolute, parent BackLeftEffector_x_link, child BackLeft_foot_cp_2_link, origin xyz=-0.09166 0.27372 -0.12195 rpy=0 0 0, axis 0 0 1, limit lower=0 upper=0 effort=15 velocity=5
- added joint BackLeft_foot_cp_3_joint: type revolute, parent BackLeftEffector_x_link, child BackLeft_foot_cp_3_link, origin xyz=-0.09166 -0.07769 -0.12195 rpy=0 0 0, axis 0 0 1, limit lower=0 upper=0 effort=15 velocity=5
- added joint BackLeft_foot_cp_4_joint: type revolute, parent BackLeftEffector_x_link, child BackLeft_foot_cp_4_link, origin xyz=0.08027 -0.07769 -0.12195 rpy=0 0 0, axis 0 0 1, limit lower=0 upper=0 effort=15 velocity=5
- added joint BackLeft_foot_endeffector_joint: type fixed, parent BackLeftEffector_x_link, child BackLeft_foot_endeffector_link, origin xyz=-0.024924 -0.097428 0.001788 rpy=0 0 0, axis 0 0 1, limit lower=-0.001 upper=0.001 effort=15 velocity=5
- added joint BackLeftshoulder_joint: type revolute, parent head_link, child BackLeftshoulder_link, origin xyz=0 0 0 rpy=0 0 0, axis 0 0 1, limit lower=-1.57 upper=1 effort=15 velocity=5
- added joint BackRightEffector_x_joint: type revolute, parent BackRightEffector_y_link, child BackRightEffector_x_link, origin xyz=0 0 0 rpy=0 0 0, axis 1 0 0, limit lower=-0.8 upper=0.6 effort=15 velocity=5
- added joint BackRightEffector_y_joint: type revolute, parent BackRightEffector_z_link, child BackRightEffector_y_link, origin xyz=0 0 0 rpy=0 0 0, axis 0 1 0, limit lower=-0.5 upper=0.5 effort=15 velocity=5
- added joint BackRightEffector_z_joint: type revolute, parent BackRightLowerLimb_link, child BackRightEffector_z_link, origin xyz=-0.4343 -0.054 -0.1597 rpy=0 0 0, axis 0 0 1, limit lower=-0.01 upper=0 effort=15 velocity=5
- added joint BackRightLimb_joint: type revolute, parent BackRightUpperLimb_x_link, child BackRightLimb_link, origin xyz=-0.4456 0.0015 0.1781 rpy=0 0 0, axis 0 1 0, limit lower=-2.4 upper=0 effort=15 velocity=5
- added joint BackRightLowerLimb_joint: type revolute, parent BackRightLimb_link, child BackRightLowerLimb_link, origin xyz=-0.3928 -0.0167 -0.3044 rpy=0 0 0, axis 0 1 0, limit lower=-2.4 upper=0 effort=15 velocity=5
- added joint BackRightUpperLimb_x_joint: type revolute, parent BackRightUpperLimb_y_link, child BackRightUpperLimb_x_link, origin xyz=0 0 0 rpy=0 0 0, axis 1 0 0, limit lower=-1.2 upper=1.57 effort=15 velocity=5
- added joint BackRightUpperLimb_y_joint: type revolute, parent BackRightUpperLimb_z_link, child BackRightUpperLimb_y_link, origin xyz=0 0 0 rpy=0 0 0, axis 0 1 0, limit lower=-1.57 upper=0.7 effort=15 velocity=5
- added joint BackRightUpperLimb_z_joint: type revolute, parent BackRightshoulder_link, child BackRightUpperLimb_z_link, origin xyz=-0.1891 0 -0.0795 rpy=0 0 0, axis 0 0 1, limit lower=-1.57 upper=1 effort=15 velocity=5
- added joint BackRight_foot_cp_1_joint: type revolute, parent BackRightEffector_x_link, child BackRight_foot_cp_1_link, origin xyz=0.08027 0.27372 -0.12195 rpy=0 0 0, axis 0 0 1, limit lower=0 upper=0 effort=15 velocity=5
- added joint BackRight_foot_cp_2_joint: type revolute, parent BackRightEffector_x_link, child BackRight_foot_cp_2_link, origin xyz=-0.09166 0.27372 -0.12195 rpy=0 0 0, axis 0 0 1, limit lower=0 upper=0 effort=15 velocity=5
- added joint BackRight_foot_cp_3_joint: type revolute, parent BackRightEffector_x_link, child BackRight_foot_cp_3_link, origin xyz=-0.09166 -0.07769 -0.12195 rpy=0 0 0, axis 0 0 1, limit lower=0 upper=0 effort=15 velocity=5
- added joint BackRight_foot_cp_4_joint: type revolute, parent BackRightEffector_x_link, child BackRight_foot_cp_4_link, origin xyz=0.08027 -0.07769 -0.12195 rpy=0 0 0, axis 0 0 1, limit lower=0 upper=0 effort=15 velocity=5
- added joint BackRight_foot_endeffector_joint: type fixed, parent BackRightEffector_x_link, child BackRight_foot_endeffector_link, origin xyz=-0.024924 -0.097428 0.001788 rpy=0 0 0, axis 0 0 1, limit lower=-0.001 upper=0.001 effort=15 velocity=5
- added joint BackRightshoulder_joint: type revolute, parent head_link, child BackRightshoulder_link, origin xyz=0 0 0 rpy=0 0 0, axis 0 0 1, limit lower=-1.57 upper=1 effort=15 velocity=5
- added joint FrontRightEffector_x_joint: type revolute, parent FrontRightEffector_y_link, child FrontRightEffector_x_link, origin xyz=0 0 0 rpy=0 0 0, axis 1 0 0, limit lower=-0.8 upper=0.6 effort=15 velocity=5
- added joint FrontRightEffector_y_joint: type revolute, parent FrontRightEffector_z_link, child FrontRightEffector_y_link, origin xyz=0 0 0 rpy=0 0 0, axis 0 1 0, limit lower=-0.5 upper=0.5 effort=15 velocity=5
- added joint FrontRightEffector_z_joint: type revolute, parent FrontRightLowerLimb_link, child FrontRightEffector_z_link, origin xyz=-0.4343 -0.054 -0.1597 rpy=0 0 0, axis 0 0 1, limit lower=-0.01 upper=0 effort=15 velocity=5
- added joint FrontRightLimb_joint: type revolute, parent FrontRightUpperLimb_x_link, child FrontRightLimb_link, origin xyz=-0.4456 0.0015 0.1781 rpy=0 0 0, axis 0 1 0, limit lower=-2.4 upper=0 effort=15 velocity=5
- added joint FrontRightLowerLimb_joint: type revolute, parent FrontRightLimb_link, child FrontRightLowerLimb_link, origin xyz=-0.3928 -0.0167 -0.3044 rpy=0 0 0, axis 0 1 0, limit lower=-2.4 upper=0 effort=15 velocity=5
- added joint FrontRightUpperLimb_x_joint: type revolute, parent FrontRightUpperLimb_y_link, child FrontRightUpperLimb_x_link, origin xyz=0 0 0 rpy=0 0 0, axis 1 0 0, limit lower=-1.2 upper=1.57 effort=15 velocity=5
- added joint FrontRightUpperLimb_y_joint: type revolute, parent FrontRightUpperLimb_z_link, child FrontRightUpperLimb_y_link, origin xyz=0 0 0 rpy=0 0 0, axis 0 1 0, limit lower=-1.57 upper=0.7 effort=15 velocity=5
- added joint FrontRightUpperLimb_z_joint: type revolute, parent FrontRightshoulder_link, child FrontRightUpperLimb_z_link, origin xyz=-0.1891 0 -0.0795 rpy=0 0 0, axis 0 0 1, limit lower=-1.57 upper=1 effort=15 velocity=5
- added joint FrontRight_foot_cp_1_joint: type revolute, parent FrontRightEffector_x_link, child FrontRight_foot_cp_1_link, origin xyz=0.08027 0.27372 -0.12195 rpy=0 0 0, axis 0 0 1, limit lower=0 upper=0 effort=15 velocity=5
- added joint FrontRight_foot_cp_2_joint: type revolute, parent FrontRightEffector_x_link, child FrontRight_foot_cp_2_link, origin xyz=-0.09166 0.27372 -0.12195 rpy=0 0 0, axis 0 0 1, limit lower=0 upper=0 effort=15 velocity=5
- added joint FrontRight_foot_cp_3_joint: type revolute, parent FrontRightEffector_x_link, child FrontRight_foot_cp_3_link, origin xyz=-0.09166 -0.07769 -0.12195 rpy=0 0 0, axis 0 0 1, limit lower=0 upper=0 effort=15 velocity=5
- added joint FrontRight_foot_cp_4_joint: type revolute, parent FrontRightEffector_x_link, child FrontRight_foot_cp_4_link, origin xyz=0.08027 -0.07769 -0.12195 rpy=0 0 0, axis 0 0 1, limit lower=0 upper=0 effort=15 velocity=5
- added joint FrontRight_foot_endeffector_joint: type fixed, parent FrontRightEffector_x_link, child FrontRight_foot_endeffector_link, origin xyz=-0.024924 -0.097428 0.001788 rpy=0 0 0, axis 0 0 1, limit lower=-0.001 upper=0.001 effort=15 velocity=5
- added joint FrontRightshoulder_joint: type revolute, parent head_link, child FrontRightshoulder_link, origin xyz=0 0 0 rpy=0 0 0, axis 0 0 1, limit lower=-1.57 upper=1 effort=15 velocity=5
- added joint Frontleft_foot_cp_1_joint: type revolute, parent FrontLeftEffector_x_link, child Frontleft_foot_cp_1_link, origin xyz=0.08027 0.27372 -0.12195 rpy=0 0 0, axis 0 0 1, limit lower=0 upper=0 effort=15 velocity=5
- added joint Frontleft_foot_cp_2_joint: type revolute, parent FrontLeftEffector_x_link, child Frontleft_foot_cp_2_link, origin xyz=-0.09166 0.27372 -0.12195 rpy=0 0 0, axis 0 0 1, limit lower=0 upper=0 effort=15 velocity=5
- added joint Frontleft_foot_cp_3_joint: type revolute, parent FrontLeftEffector_x_link, child Frontleft_foot_cp_3_link, origin xyz=-0.09166 -0.07769 -0.12195 rpy=0 0 0, axis 0 0 1, limit lower=0 upper=0 effort=15 velocity=5
- added joint Frontleft_foot_cp_4_joint: type revolute, parent FrontLeftEffector_x_link, child Frontleft_foot_cp_4_link, origin xyz=0.08027 -0.07769 -0.12195 rpy=0 0 0, axis 0 0 1, limit lower=0 upper=0 effort=15 velocity=5
- added joint Frontleft_foot_endeffector_joint: type fixed, parent FrontLeftEffector_x_link, child Frontleft_foot_endeffector_link, origin xyz=-0.024924 -0.097428 0.001788 rpy=0 0 0, axis 0 0 1, limit lower=-0.001 upper=0.001 effort=15 velocity=5
- added joint MiddleRightEffector_x_joint: type revolute, parent MiddleRightEffector_y_link, child MiddleRightEffector_x_link, origin xyz=0 0 0 rpy=0 0 0, axis 1 0 0, limit lower=-0.8 upper=0.6 effort=15 velocity=5
- added joint MiddleRightEffector_y_joint: type revolute, parent MiddleRightEffector_z_link, child MiddleRightEffector_y_link, origin xyz=0 0 0 rpy=0 0 0, axis 0 1 0, limit lower=-0.5 upper=0.5 effort=15 velocity=5
- added joint MiddleRightEffector_z_joint: type revolute, parent MiddleRightLowerLimb_link, child MiddleRightEffector_z_link, origin xyz=-0.4343 -0.054 -0.1597 rpy=0 0 0, axis 0 0 1, limit lower=-0.01 upper=0 effort=15 velocity=5
- added joint MiddleRightLimb_joint: type revolute, parent MiddleRightUpperLimb_x_link, child MiddleRightLimb_link, origin xyz=-0.4456 0.0015 0.1781 rpy=0 0 0, axis 0 1 0, limit lower=-2.4 upper=0 effort=15 velocity=5
- added joint MiddleRightLowerLimb_joint: type revolute, parent MiddleRightLimb_link, child MiddleRightLowerLimb_link, origin xyz=-0.3928 -0.0167 -0.3044 rpy=0 0 0, axis 0 1 0, limit lower=-2.4 upper=0 effort=15 velocity=5
- added joint MiddleRightUpperLimb_x_joint: type revolute, parent MiddleRightUpperLimb_y_link, child MiddleRightUpperLimb_x_link, origin xyz=0 0 0 rpy=0 0 0, axis 1 0 0, limit lower=-1.2 upper=1.57 effort=15 velocity=5
- added joint MiddleRightUpperLimb_y_joint: type revolute, parent MiddleRightUpperLimb_z_link, child MiddleRightUpperLimb_y_link, origin xyz=0 0 0 rpy=0 0 0, axis 0 1 0, limit lower=-1.57 upper=0.7 effort=15 velocity=5
- added joint MiddleRightUpperLimb_z_joint: type revolute, parent MiddleRightshoulder_link, child MiddleRightUpperLimb_z_link, origin xyz=-0.1891 0 -0.0795 rpy=0 0 0, axis 0 0 1, limit lower=-1.57 upper=1 effort=15 velocity=5
- added joint MiddleRight_foot_cp_1_joint: type revolute, parent MiddleRightEffector_x_link, child MiddleRight_foot_cp_1_link, origin xyz=0.08027 0.27372 -0.12195 rpy=0 0 0, axis 0 0 1, limit lower=0 upper=0 effort=15 velocity=5
- added joint MiddleRight_foot_cp_2_joint: type revolute, parent MiddleRightEffector_x_link, child MiddleRight_foot_cp_2_link, origin xyz=-0.09166 0.27372 -0.12195 rpy=0 0 0, axis 0 0 1, limit lower=0 upper=0 effort=15 velocity=5
- added joint MiddleRight_foot_cp_3_joint: type revolute, parent MiddleRightEffector_x_link, child MiddleRight_foot_cp_3_link, origin xyz=-0.09166 -0.07769 -0.12195 rpy=0 0 0, axis 0 0 1, limit lower=0 upper=0 effort=15 velocity=5
- added joint MiddleRight_foot_cp_4_joint: type revolute, parent MiddleRightEffector_x_link, child MiddleRight_foot_cp_4_link, origin xyz=0.08027 -0.07769 -0.12195 rpy=0 0 0, axis 0 0 1, limit lower=0 upper=0 effort=15 velocity=5
- added joint MiddleRight_foot_endeffector_joint: type fixed, parent MiddleRightEffector_x_link, child MiddleRight_foot_endeffector_link, origin xyz=-0.024924 -0.097428 0.001788 rpy=0 0 0, axis 0 0 1, limit lower=-0.001 upper=0.001 effort=15 velocity=5
- added joint MiddleRightshoulder_joint: type revolute, parent head_link, child MiddleRightshoulder_link, origin xyz=0 0 0 rpy=0 0 0, axis 0 0 1, limit lower=-1.57 upper=1 effort=15 velocity=5
- added joint frontleftshoulder_joint: type revolute, parent head_link, child frontleftshoulder_link, origin xyz=0 0 0 rpy=0 0 0, axis 0 0 1, limit lower=-1.57 upper=1 effort=15 velocity=5
- added joint middleleftshoulder_joint: type revolute, parent head_link, child middleleftshoulder_link, origin xyz=0 0 0 rpy=0 0 0, axis 0 0 1, limit lower=-1.57 upper=1 effort=15 velocity=5
- joint FrontLeftEffector_z_joint: origin xyz=-0.3452 0.3029 -0.166 rpy=0 0 0 -> xyz=-0.4343 -0.054 -0.1597 rpy=0 0 0
- joint FrontLeftLimb_joint: axis 1 0 0 -> 0 1 0; origin xyz=-0.3344 0.3178 0.1886 rpy=0 0 0 -> xyz=-0.4456 0.0015 0.1781 rpy=0 0 0
- joint FrontLeftLowerLimb_joint: axis 1 0 0 -> 0 1 0; origin xyz=-0.2936 0.2729 -0.2964 rpy=0 0 0 -> xyz=-0.3928 -0.0167 -0.3044 rpy=0 0 0
- joint FrontLeftUpperLimb_z_joint: origin xyz=-0.1619 0.1824 -0.0689 rpy=0 0 0 -> xyz=-0.1891 0 -0.0795 rpy=0 0 0; parent head_link -> frontleftshoulder_link

Commit message: weird effector not fully aligned

File: spider/model/spider.urdf (robot description, URDF)
Before this commit: robot rocketbox_male, 95 links, 94 joints
Joints:
- joint Frontleft_foot_cp_1_joint: parent FrontLeftEffector_x_link -> Frontleft_foot_endeffector_link
- joint Frontleft_foot_cp_2_joint: parent FrontLeftEffector_x_link -> Frontleft_foot_endeffector_link
- joint Frontleft_foot_cp_3_joint: parent FrontLeftEffector_x_link -> Frontleft_foot_endeffector_link
- joint Frontleft_foot_cp_4_joint: parent FrontLeftEffector_x_link -> Frontleft_foot_endeffector_link
- joint Frontleft_foot_endeffector_joint: origin xyz=-0.024924 -0.097428 0.001788 rpy=0 0 0 -> xyz=-0.1086 -0.0059 -0.0138 rpy=0 0 0; type fixed -> revolute
