Commit message: fixed contact points locations

File: spider/model/spider.urdf (robot description, URDF)
Before this commit: robot rocketbox_male, 95 links, 94 joints
Joints:
- joint BackLeft_foot_cp_1_joint: origin xyz=0.08027 0.27372 -0.12195 rpy=0 0 0 -> xyz=-0.05 0.02 -0.005 rpy=0 0 0
- joint BackLeft_foot_cp_2_joint: origin xyz=-0.09166 0.27372 -0.12195 rpy=0 0 0 -> xyz=-0.12 0.02 -0.005 rpy=0 0 0
- joint BackLeft_foot_cp_3_joint: origin xyz=-0.09166 -0.07769 -0.12195 rpy=0 0 0 -> xyz=-0.12 -0.08 -0.005 rpy=0 0 0
- joint BackLeft_foot_cp_4_joint: origin xyz=0.08027 -0.07769 -0.12195 rpy=0 0 0 -> xyz=-0.05 -0.08 -0.005 rpy=0 0 0
- joint BackRight_foot_cp_1_joint: origin xyz=0.08027 0.27372 -0.12195 rpy=0 0 0 -> xyz=-0.05 0.02 -0.005 rpy=0 0 0
- joint BackRight_foot_cp_2_joint: origin xyz=-0.09166 0.27372 -0.12195 rpy=0 0 0 -> xyz=-0.12 0.02 -0.005 rpy=0 0 0
- joint BackRight_foot_cp_3_joint: origin xyz=-0.09166 -0.07769 -0.12195 rpy=0 0 0 -> xyz=-0.12 -0.08 -0.005 rpy=0 0 0
- joint BackRight_foot_cp_4_joint: origin xyz=0.08027 -0.07769 -0.12195 rpy=0 0 0 -> xyz=-0.05 -0.08 -0.005 rpy=0 0 0
- joint FrontRight_foot_cp_1_joint: origin xyz=0.08027 0.27372 -0.12195 rpy=0 0 0 -> xyz=-0.05 0.02 -0.005 rpy=0 0 0
- joint FrontRight_foot_cp_2_joint: origin xyz=-0.09166 0.27372 -0.12195 rpy=0 0 0 -> xyz=-0.12 0.02 -0.005 rpy=0 0 0
- joint FrontRight_foot_cp_3_joint: origin xyz=-0.09166 -0.07769 -0.12195 rpy=0 0 0 -> xyz=-0.12 -0.08 -0.005 rpy=0 0 0
- joint FrontRight_foot_cp_4_joint: origin xyz=0.08027 -0.07769 -0.12195 rpy=0 0 0 -> xyz=-0.05 -0.08 -0.005 rpy=0 0 0
- joint Frontleft_foot_cp_1_joint: origin xyz=0.08027 0.27372 -0.12195 rpy=0 0 0 -> xyz=0.08027 0.27372 0 rpy=0 0 0
- joint Frontleft_foot_cp_2_joint: origin xyz=-0.09166 0.27372 -0.12195 rpy=0 0 0 -> xyz=-0.09166 0.27372 0 rpy=0 0 0
- joint Frontleft_foot_cp_3_joint: origin xyz=-0.09166 -0.07769 -0.12195 rpy=0 0 0 -> xyz=-0.09166 -0.07769 0 rpy=0 0 0
- joint Frontleft_foot_cp_4_joint: origin xyz=0.08027 -0.07769 -0.12195 rpy=0 0 0 -> xyz=0.08027 -0.07769 0 rpy=0 0 0
- joint MiddleRight_foot_cp_1_joint: origin xyz=0.08027 0.27372 -0.12195 rpy=0 0 0 -> xyz=-0.05 0.02 -0.005 rpy=0 0 0
- joint MiddleRight_foot_cp_2_joint: origin xyz=-0.09166 0.27372 -0.12195 rpy=0 0 0 -> xyz=-0.12 0.02 -0.005 rpy=0 0 0
- joint MiddleRight_foot_cp_3_joint: origin xyz=-0.09166 -0.07769 -0.12195 rpy=0 0 0 -> xyz=-0.12 -0.08 -0.005 rpy=0 0 0
- joint MiddleRight_foot_cp_4_joint: origin xyz=0.08027 -0.07769 -0.12195 rpy=0 0 0 -> xyz=-0.05 -0.08 -0.005 rpy=0 0 0
- joint Middleleft_foot_cp_1_joint: origin xyz=0.08027 0.27372 -0.12195 rpy=0 0 0 -> xyz=-0.05 0.02 -0.005 rpy=0 0 0
- joint Middleleft_foot_cp_2_joint: origin xyz=-0.09166 0.27372 -0.12195 rpy=0 0 0 -> xyz=-0.12 0.02 -0.005 rpy=0 0 0
- joint Middleleft_foot_cp_3_joint: origin xyz=-0.09166 -0.07769 -0.12195 rpy=0 0 0 -> xyz=-0.12 -0.08 -0.005 rpy=0 0 0
- joint Middleleft_foot_cp_4_joint: origin xyz=0.08027 -0.07769 -0.12195 rpy=0 0 0 -> xyz=-0.05 -0.08 -0.005 rpy=0 0 0

Commit message: final bug fixes in urdf. onto dual shapes

File: spider/model/spider.urdf (robot description, URDF)
Before this commit: robot rocketbox_male, 95 links, 94 joints
Joints:
- joint Frontleft_foot_cp_1_joint: origin xyz=0.08027 0.27372 0 rpy=0 0 0 -> xyz=-0.05 0.02 -0.005 rpy=0 0 0; parent Frontleft_foot_endeffector_link -> FrontLeftEffector_x_link
- joint Frontleft_foot_cp_2_joint: origin xyz=-0.09166 0.27372 0 rpy=0 0 0 -> xyz=-0.12 0.02 -0.005 rpy=0 0 0; parent Frontleft_foot_endeffector_link -> FrontLeftEffector_x_link
- joint Frontleft_foot_cp_3_joint: origin xyz=-0.09166 -0.07769 0 rpy=0 0 0 -> xyz=-0.12 -0.08 -0.005 rpy=0 0 0; parent Frontleft_foot_endeffector_link -> FrontLeftEffector_x_link
- joint Frontleft_foot_cp_4_joint: origin xyz=0.08027 -0.07769 0 rpy=0 0 0 -> xyz=-0.05 -0.08 -0.005 rpy=0 0 0; parent Frontleft_foot_endeffector_link -> FrontLeftEffector_x_link

Commit message: final urdf ?

File: spider/model/spider.urdf (robot description, URDF)
Before this commit: robot rocketbox_male, 95 links, 94 joints
Joints:
- joint BackLeft_foot_endeffector_joint: type fixed -> revolute
- joint BackRight_foot_endeffector_joint: type fixed -> revolute
- joint FrontRight_foot_endeffector_joint: type fixed -> revolute
- joint MiddleRight_foot_endeffector_joint: type fixed -> revolute
- joint Middleleft_foot_endeffector_joint: type fixed -> revolute
