Commit message: adding obj models

File: rami/model/human_rami.urdf (robot description, URDF)
Before this commit: robot rocketbox_male, 64 links, 63 joints
Links:
- removed link HEad_x_link
- removed link HEad_y_link
- removed link HEad_z_link
- added link LeftHandendsite_x_link
- added link LeftHandendsite_y_link
- added link LeftHandendsite_z_link
- added link LeftToesendsite_x_link
- added link LeftToesendsite_y_link
- added link LeftToesendsite_z_link
- added link RightHandendsite_x_link
- added link RightHandendsite_y_link
- added link RightHandendsite_z_link
- added link RightToesendsite_x_link
- added link RightToesendsite_y_link
- added link RightToesendsite_z_link
- added link head_x_link; collision mesh filename=../rami/model/head.obj; visual mesh filename=../rami/model/head.obj
- added link head_y_link
- added link head_z_link
- added link headendsite_x_link
- added link headendsite_y_link
- added link headendsite_z_link
Joints:
- removed joint HEad_x_joint
- removed joint HEad_y_joint
- removed joint HEad_z_joint
- added joint LeftHandendsite_x_joint: type revolute, parent LeftHandendsite_y_link, child LeftHandendsite_x_link, origin xyz=0 0 0 rpy=0 0 0, axis 1 0 0, limit lower=-3.14 upper=3.14 effort=10000 velocity=0.6
- added joint LeftHandendsite_y_joint: type revolute, parent LeftHandendsite_z_link, child LeftHandendsite_y_link, origin xyz=0 0 0 rpy=0 0 0, axis 0 1 0, limit lower=-3.14 upper=3.14 effort=10000 velocity=0.6
- added joint LeftHandendsite_z_joint: type revolute, parent LeftHand_x_link, child LeftHandendsite_z_link, origin xyz=0.167443 -0.006 0.0150291 rpy=0 0 0, axis 0 0 1, limit lower=-3.14 upper=3.14 effort=10000 velocity=0.6
- added joint LeftToesendsite_x_joint: type revolute, parent LeftToesendsite_y_link, child LeftToesendsite_x_link, origin xyz=0 0 0 rpy=0 0 0, axis 1 0 0, limit lower=-3.14 upper=3.14 effort=10000 velocity=0.6
- added joint LeftToesendsite_y_joint: type revolute, parent LeftToesendsite_z_link, child LeftToesendsite_y_link, origin xyz=0 0 0 rpy=0 0 0, axis 0 1 0, limit lower=-3.14 upper=3.14 effort=10000 velocity=0.6
- added joint LeftToesendsite_z_joint: type revolute, parent LeftToes_x_link, child LeftToesendsite_z_link, origin xyz=0.0008 -0.0004745 0.0977979 rpy=0 0 0, axis 0 0 1, limit lower=-3.14 upper=3.14 effort=10000 velocity=0.6
- added joint RightHandendsite_x_joint: type revolute, parent RightHandendsite_y_link, child RightHandendsite_x_link, origin xyz=0 0 0 rpy=0 0 0, axis 1 0 0, limit lower=-3.14 upper=3.14 effort=10000 velocity=0.6
- added joint RightHandendsite_y_joint: type revolute, parent RightHandendsite_z_link, child RightHandendsite_y_link, origin xyz=0 0 0 rpy=0 0 0, axis 0 1 0, limit lower=-3.14 upper=3.14 effort=10000 velocity=0.6
- added joint RightHandendsite_z_joint: type revolute, parent RightHand_x_link, child RightHandendsite_z_link, origin xyz=-0.166312 -0.006 0.0150291 rpy=0 0 0, axis 0 0 1, limit lower=-3.14 upper=3.14 effort=10000 velocity=0.6
- added joint RightToesendsite_x_joint: type revolute, parent RightToesendsite_y_link, child RightToesendsite_x_link, origin xyz=0 0 0 rpy=0 0 0, axis 1 0 0, limit lower=-3.14 upper=3.14 effort=10000 velocity=0.6
- added joint RightToesendsite_y_joint: type revolute, parent RightToesendsite_z_link, child RightToesendsite_y_link, origin xyz=0 0 0 rpy=0 0 0, axis 0 1 0, limit lower=-3.14 upper=3.14 effort=10000 velocity=0.6
- added joint RightToesendsite_z_joint: type revolute, parent RightToes_x_link, child RightToesendsite_z_link, origin xyz=-0.0008 -0.0013745 0.0977979 rpy=0 0 0, axis 0 0 1, limit lower=-3.14 upper=3.14 effort=10000 velocity=0.6
- added joint head_x_joint: type revolute, parent head_y_link, child head_x_link, origin xyz=0 0 0 rpy=0 0 0, axis 1 0 0, limit lower=-3.14 upper=3.14 effort=10000 velocity=0.6
- added joint head_y_joint: type revolute, parent head_z_link, child head_y_link, origin xyz=0 0 0 rpy=0 0 0, axis 0 1 0, limit lower=-3.14 upper=3.14 effort=10000 velocity=0.6
- added joint head_z_joint: type revolute, parent Spine1_x_link, child head_z_link, origin xyz=0 0.0873416 0.0001134 rpy=0 0 0, axis 0 0 1, limit lower=-3.14 upper=3.14 effort=10000 velocity=0.6
- added joint headendsite_x_joint: type revolute, parent headendsite_y_link, child headendsite_x_link, origin xyz=0 0 0 rpy=0 0 0, axis 1 0 0, limit lower=-3.14 upper=3.14 effort=10000 velocity=0.6
- added joint headendsite_y_joint: type revolute, parent headendsite_z_link, child headendsite_y_link, origin xyz=0 0 0 rpy=0 0 0, axis 0 1 0, limit lower=-3.14 upper=3.14 effort=10000 velocity=0.6
- added joint headendsite_z_joint: type revolute, parent head_x_link, child headendsite_z_link, origin xyz=-0.0029 0.127742 0.0251395 rpy=0 0 0, axis 0 0 1, limit lower=-3.14 upper=3.14 effort=10000 velocity=0.6
- joint LeftArm_z_joint: origin xyz=0.102827 -3.37999e-05 0.00322123 rpy=0 0 0 -> xyz=0.102827 -3.38e-05 0.0032212 rpy=0 0 0
- joint LeftFoot_z_joint: origin xyz=-0.00253549 -0.420924 -0.0146059 rpy=0 0 0 -> xyz=-0.0025355 -0.420924 -0.0146059 rpy=0 0 0
- joint LeftForeArm_z_joint: origin xyz=0.262597 0.00099144 -0.0142434 rpy=0 0 0 -> xyz=0.327669 0.0009914 -0.0142434 rpy=0 0 0
- joint LeftHand_z_joint: origin xyz=0.134179 -0.00600076 0.0150291 rpy=0 0 0 -> xyz=0.275643 0.0008536 0.0102216 rpy=0 0 0
- joint LeftShoulder1_z_joint: origin xyz=0.0899 -0.00362252 -0.0022 rpy=0 0 0 -> xyz=0.0899 -0.0036225 -0.0022 rpy=0 0 0
- joint LeftToes_z_joint: origin xyz=0.0008 -0.00047448 0.0977979 rpy=0 0 0 -> xyz=-0.0004 -0.0441509 0.084991 rpy=0 0 0
- joint LeftUpLeg_z_joint: origin xyz=0.089458 -0.0866707 0.00101652 rpy=0 0 0 -> xyz=0.089458 -0.0866707 0.0010165 rpy=0 0 0
- joint RightArm_z_joint: origin xyz=-0.102827 -3.38e-05 0.00322123 rpy=0 0 0 -> xyz=-0.102827 -3.38e-05 0.0032212 rpy=0 0 0
- joint RightFoot_z_joint: origin xyz=0.00253549 -0.420924 -0.0146059 rpy=0 0 0 -> xyz=0.0025355 -0.420924 -0.0146059 rpy=0 0 0
- joint RightForeArm_z_joint: origin xyz=-0.26364 0.00099144 -0.0142434 rpy=0 0 0 -> xyz=-0.328971 0.0009914 -0.0142434 rpy=0 0 0
- joint RightHand_z_joint: origin xyz=-0.133273 -0.00600075 0.0150291 rpy=0 0 0 -> xyz=-0.274921 0.0008536 0.0102216 rpy=0 0 0
- joint RightShoulder_z_joint: origin xyz=-0.0899 -0.00362252 -0.0022 rpy=0 0 0 -> xyz=-0.0899 -0.0036225 -0.0022 rpy=0 0 0
- joint RightToes_z_joint: origin xyz=-0.0008 -0.00137448 0.0977979 rpy=0 0 0 -> xyz=0.0004 -0.0441509 0.084991 rpy=0 0 0
- joint RightUpLeg_z_joint: origin xyz=-0.089458 -0.0866707 0.00101652 rpy=0 0 0 -> xyz=-0.089458 -0.0866707 0.0010165 rpy=0 0 0
- joint Spine1_z_joint: origin xyz=0 0.256574 0.00127663 rpy=0 0 0 -> xyz=0 0.256574 0.0012766 rpy=0 0 0
- joint Spine_z_joint: origin xyz=0 0.118905 0 rpy=0 0 0 -> xyz=0 0.118905 -0 rpy=0 0 0

Commit message: bvh to urdf complete

File: rami/model/human_rami.urdf (robot description, URDF)
Before this commit: robot rocketbox_male, 79 links, 78 joints
Links:
- link LeftHandendsite_x_link: geometry collision mesh filename=../rami/model/LeftHandendsite.obj; visual mesh filename=../rami/model/LeftHandendsite.obj
- link LeftToesendsite_x_link: geometry collision mesh filename=../rami/model/LeftToesendsite.obj; visual mesh filename=../rami/model/LeftToesendsite.obj
- link RightHandendsite_x_link: geometry collision mesh filename=../rami/model/RightHandendsite.obj; visual mesh filename=../rami/model/RightHandendsite.obj
- link RightToesendsite_x_link: geometry collision mesh filename=../rami/model/RightToesendsite.obj; visual mesh filename=../rami/model/RightToesendsite.obj
- link headendsite_x_link: geometry collision mesh filename=../rami/model/headendsite.obj; visual mesh filename=../rami/model/headendsite.obj
